Commit message: feat: add Piper expert policy and ACT demo collection

File: robot_assets/piper_l/piper_l_gripper_d435.urdf (robot description, URDF)
Before this commit: robot agx_arm, 15 links, 14 joints
Links:
- added link grasp_tcp
Joints:
- added joint grasp_tcp_joint: type fixed, parent link6, child grasp_tcp, origin xyz=0 0 0.0593 rpy=0 0 0

Commit message: fix: stabilize Piper expert data collection

File: robot_assets/piper_l/piper_l_gripper_d435.urdf (robot description, URDF)
Before this commit: robot agx_arm, 16 links, 15 joints
Joints:
- joint grasp_tcp_joint: origin xyz=0 0 0.0593 rpy=0 0 0 -> xyz=0 0 0.1358 rpy=0 0 0

Commit message: Build planning-only dual-arm validation platform

File: robot_assets/piper_l/piper_l_gripper_d435.urdf (robot description, URDF)
Before this commit: robot agx_arm, 15 links, 14 joints
Joints:
- joint joint4: limit lower=-1.7453292 upper=1.7453292 effort=100 velocity=5 -> lower=-2.2165681 upper=2.2165681 effort=100 velocity=5
- joint joint5: limit lower=-1.2217304 upper=1.2217304 effort=100 velocity=5 -> lower=-1.5620696 upper=1.5620696 effort=100 velocity=5

Commit message: Add formal Piper execution chain baseline

File: robot_assets/piper_l/piper_l_gripper_d435.urdf (robot description, URDF)
Before this commit: robot agx_arm, 15 links, 14 joints
Joints:
- joint joint4: limit lower=-2.2165681 upper=2.2165681 effort=100 velocity=5 -> lower=-1.7453292 upper=1.7453292 effort=100 velocity=5
- joint joint5: limit lower=-1.5620696 upper=1.5620696 effort=100 velocity=5 -> lower=-1.2217304 upper=1.2217304 effort=100 velocity=5
